Commit message: fix(urdf): drop meaningless <axis> on the fixed gripper_frame_joint
ikpy warns "Joint gripper_frame_joint is of type: fixed, but has an 'axis'
attribute defined ... this axis is ignored" on every chain load. The axis is a
no-op on a fixed joint (ikpy already ignores it), so removing the line silences
the warning at its source with zero change to FK/IK. Verified: 0 axis warnings,
FK and solve_ik unchanged.

Co-Authored-By: Claude Opus 4.8 <noreply@anthropic.com>

File: assets/so101/so101_new_calib.urdf (robot description, URDF)
Before this commit: robot so101_new_calib, 8 links, 7 joints
Joints:
- joint gripper_frame_joint: axis 0 0 0 -> (none)
